File: 2364-27512-Adapter.kicad_pcb (KiCad board)
At the start: 2 copper layers, 26.7 x 39.4 mm, 4 parts, among them U1 2364, U2 27512

Commit message: Add files via upload
Parts:
- removed REF** (x2): VIA_0.6mm, C64:VIA_0.6mm
Changed lines of the file:
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@@
     (area 135.89 99.06 171.450001 144.780001)
     (thickness 1.6)
-    (drawings 10)
+    (drawings 9)
     (tracks 33)
     (zones 0)
-    (modules 4)
+    (modules 2)
     (nets 25)
   )
@@
     (rev 0.10)
     (company VintageProject)
-    (comment 1 "Use for C64 ROM replacement")
+    (comment 1 "Use for C64 ROM replacements")
   )
   (layers
@@
     (46 B.CrtYd user)
     (47 F.CrtYd user)
-    (48 B.Fab user)
-    (49 F.Fab user)
+    (48 B.Fab user hide)
+    (49 F.Fab user hide)
   )
   (setup
@@
     (visible_elements 7FFFFFFF)
     (pcbplotparams
-      (layerselection 0x20020_00000001)
-      (usegerberextensions false)
-      (excludeedgelayer false)
+      (layerselection 0x010f0_80000001)
+      (usegerberextensions true)
+      (excludeedgelayer true)
       (linewidth 0.100000)
       (plotframeref false)
@@
       (padsonsilk false)
       (subtractmaskfromsilk false)
-      (outputformat 4)
+      (outputformat 1)
       (mirror false)
-      (drillshape 1)
+      (drillshape 0)
       (scaleselection 1)
-      (outputdirectory ""))
+      (outputdirectory "D:/OneDrive - Thilo Niewöhner/2.29-KiCad/2364-27512-Adapter/gerber/"))
   )
   (net 0 "")
@@
     )
   )
-  (module C64:VIA_0.6mm (layer F.Cu)
-    (at 153.67 111.76)
-    (fp_text reference REF** (at 0 0.5) (layer F.SilkS)
-      (effects (font (size 0.127 0.127) (thickness 0.01)))
-    )
-    (fp_text value VIA_0.6mm (at 0 -0.5) (layer F.Fab)
-      (effects (font (size 0.2 0.2) (thickness 0.01)))
-    )
-  )
-  (module C64:VIA_0.6mm (layer F.Cu)
-    (at 153.67 111.76)
-    (fp_text reference REF** (at 0 0.5) (layer F.SilkS)
-      (effects (font (size 0.127 0.127) (thickness 0.01)))
-    )
-    (fp_text value VIA_0.6mm (at 0 -0.5) (layer F.Fab)
-      (effects (font (size 0.2 0.2) (thickness 0.01)))
-    )
-  )
-  (gr_text "2364 to 27512 Adapter v0.10" (at 142.24 139.7) (layer F.Fab)
+  (gr_text "2364 to 27512 Adapter v0.10" (at 142.24 139.7) (layer F.SilkS)
     (effects (font (size 1 1) (thickness 0.1)) (justify left))
   )
@@
     (effects (font (size 1 1.5) (thickness 0.1)) (justify left mirror))
   )
-  (target plus (at 140.97 101.6) (size 5) (width 0.15) (layer Edge.Cuts))
   (gr_line (start 142.24 101.6) (end 156.21 101.6) (angle 90) (layer Edge.Cuts) (width 0.15))
   (gr_line (start 140.97 101.6) (end 142.24 101.6) (angle 90) (layer Edge.Cuts) (width 0.15))

Commit message: Minor tweaks
Parts:
- added G***: LOGO_VintageProject_B.SilkS, Thilo_Lib:LOGO_VintageProject_B.SilkS, F.Cu at (152.9, 112.8)
Connections:
- net Net-(U1-Pad1) renamed /A7
- net Net-(U1-Pad10) renamed /D1
- net Net-(U1-Pad11) renamed /D2
- net Net-(U1-Pad13) renamed /D3
- net Net-(U1-Pad14) renamed /D4
- net Net-(U1-Pad15) renamed /D5
- net Net-(U1-Pad16) renamed /D6
- net Net-(U1-Pad17) renamed /D7
- net Net-(U1-Pad18) renamed /A11
- net Net-(U1-Pad19) renamed /A10
- net Net-(U1-Pad2) renamed /A6
- net Net-(U1-Pad20) renamed /CE
- net Net-(U1-Pad21) renamed /A12
- net Net-(U1-Pad22) renamed /A9
- net Net-(U1-Pad23) renamed /A8
- net Net-(U1-Pad3) renamed /A5
- net Net-(U1-Pad4) renamed /A4
- net Net-(U1-Pad5) renamed /A3
- net Net-(U1-Pad6) renamed /A2
- net Net-(U1-Pad7) renamed /A1
- net Net-(U1-Pad8) renamed /A0
- net Net-(U1-Pad9) renamed /D0
